Commit message: add steering control

File: src/mini_car_description/urdf/mini_car.urdf.xacro (robot description, xacro)
@@ -16,4 +16,9 @@
   <xacro:property name="lidar_radius" value="0.045"/>
   <xacro:property name="lidar_height" value="0.04"/>
+  <!-- Ackermann drive parameters -->
+  <xacro:property name="wheel_base" value="${front_axle_x - rear_axle_x}"/>
+  <xacro:property name="track_width" value="${wheel_y * 2.0}"/>
+  <xacro:property name="max_steer_angle" value="0.6"/>
+  <xacro:property name="max_speed" value="2.0"/>
   <!-- Derived values -->
   <xacro:property
@@ -147,5 +152,6 @@
     <origin xyz="${front_axle_x} ${wheel_y} ${wheel_joint_z}" rpy="0 0 0"/>
     <axis xyz="0 0 1"/>
-    <limit lower="-0.6" upper="0.6" effort="10.0" velocity="1.0"/>
+    <limit lower="${-max_steer_angle}" upper="${max_steer_angle}" effort="100.0" velocity="2.0"/>
+    <dynamics damping="1.0" friction="0.1"/>
   </joint>
   <joint name="front_left_wheel_joint" type="continuous">
@@ -154,4 +160,5 @@
     <origin xyz="0 0 0" rpy="0 0 0"/>
     <axis xyz="0 1 0"/>
+    <dynamics damping="0.1" friction="0.0"/>
   </joint>
   <!-- ========================= -->
@@ -165,5 +172,6 @@
     <origin xyz="${front_axle_x} ${-wheel_y} ${wheel_joint_z}" rpy="0 0 0"/>
     <axis xyz="0 0 1"/>
-    <limit lower="-0.6" upper="0.6" effort="10.0" velocity="1.0"/>
+    <limit lower="${-max_steer_angle}" upper="${max_steer_angle}" effort="100.0" velocity="2.0"/>
+    <dynamics damping="1.0" friction="0.1"/>
   </joint>
   <joint name="front_right_wheel_joint" type="continuous">
@@ -172,4 +180,5 @@
     <origin xyz="0 0 0" rpy="0 0 0"/>
     <axis xyz="0 1 0"/>
+    <dynamics damping="0.1" friction="0.0"/>
   </joint>
   <!-- ========================= -->
@@ -182,4 +191,5 @@
     <origin xyz="${rear_axle_x} ${wheel_y} ${wheel_joint_z}" rpy="0 0 0"/>
     <axis xyz="0 1 0"/>
+    <dynamics damping="0.1" friction="0.0"/>
   </joint>
   <!-- ========================= -->
@@ -192,4 +202,5 @@
     <origin xyz="${rear_axle_x} ${-wheel_y} ${wheel_joint_z}" rpy="0 0 0"/>
     <axis xyz="0 1 0"/>
+    <dynamics damping="0.1" friction="0.0"/>
   </joint>
   <!-- ========================= -->
@@ -230,3 +241,133 @@
       rpy="0 0 0"/>
   </joint>
+  <!-- ========================= -->
+  <!-- Virtual steering wheel -->
+  <!-- Used by gazebo_ros_ackermann_drive plugin -->
+  <!-- ========================= -->
+  <link name="steering_wheel_link">
+    <visual>
+      <origin xyz="0 0 0" rpy="1.5708 0 0"/>
+      <geometry>
+        <cylinder radius="0.04" length="0.01"/>
+      </geometry>
+      <material name="yellow"/>
+    </visual>
+    <collision>
+      <origin xyz="0 0 0" rpy="1.5708 0 0"/>
+      <geometry>
+        <cylinder radius="0.04" length="0.01"/>
+      </geometry>
+    </collision>
+    <inertial>
+      <origin xyz="0 0 0" rpy="0 0 0"/>
+      <mass value="0.05"/>
+      <inertia
+        ixx="0.00005"
+        ixy="0.0"
+        ixz="0.0"
+        iyy="0.00005"
+        iyz="0.0"
+        izz="0.00005"/>
+    </inertial>
+  </link>
+  <joint name="steering_wheel_joint" type="revolute">
+    <parent link="base_link"/>
+    <child link="steering_wheel_link"/>
+    <origin xyz="0.12 0 0.08" rpy="0 0 0"/>
+    <axis xyz="0 0 1"/>
+    <limit lower="-7.85" upper="7.85" effort="10.0" velocity="5.0"/>
+    <dynamics damping="0.1" friction="0.0"/>
+  </joint>
+  <!-- ========================= -->
+  <!-- Gazebo visual/friction properties -->
+  <!-- ========================= -->
+  <gazebo reference="base_link">
+    <material>Gazebo/Blue</material>
+  </gazebo>
+  <gazebo reference="front_left_steering_link">
+    <material>Gazebo/Yellow</material>
+  </gazebo>
+  <gazebo reference="front_right_steering_link">
+    <material>Gazebo/Yellow</material>
+  </gazebo>
+  <gazebo reference="front_left_wheel_link">
+    <material>Gazebo/Grey</material>
+    <mu1>1.5</mu1>
+    <mu2>1.5</mu2>
+    <kp>1000000.0</kp>
+    <kd>100.0</kd>
+  </gazebo>
+  <gazebo reference="front_right_wheel_link">
+    <material>Gazebo/Grey</material>
+    <mu1>1.5</mu1>
+    <mu2>1.5</mu2>
+    <kp>1000000.0</kp>
+    <kd>100.0</kd>
+  </gazebo>
+  <gazebo reference="rear_left_wheel_link">
+    <material>Gazebo/Grey</material>
+    <mu1>1.5</mu1>
+    <mu2>1.5</mu2>
+    <kp>1000000.0</kp>
+    <kd>100.0</kd>
+  </gazebo>
+  <gazebo reference="rear_right_wheel_link">
+    <material>Gazebo/Grey</material>
+    <mu1>1.5</mu1>
+    <mu2>1.5</mu2>
+    <kp>1000000.0</kp>
+    <kd>100.0</kd>
+  </gazebo>
+  <gazebo reference="lidar_link">
+    <material>Gazebo/Red</material>
+  </gazebo>
+  <gazebo reference="steering_wheel_link">
+    <material>Gazebo/Yellow</material>
+  </gazebo>
+  <!-- ========================= -->
+  <!-- ros2_control configuration -->
+  <!-- ========================= -->
+  <ros2_control name="GazeboSimSystem" type="system">
+    <hardware>
+      <plugin>gz_ros2_control/GazeboSimSystem</plugin>
+    </hardware>
+    <!-- Front steering joints: position control -->
+    <joint name="front_left_steering_joint">
+      <command_interface name="position">
+        <param name="min">-0.6</param>
+        <param name="max">0.6</param>
+      </command_interface>
+      <state_interface name="position"/>
+      <state_interface name="velocity"/>
+    </joint>
+    <joint name="front_right_steering_joint">
+      <command_interface name="position">
+        <param name="min">-0.6</param>
+        <param name="max">0.6</param>
+      </command_interface>
+      <state_interface name="position"/>
+      <state_interface name="velocity"/>
+    </joint>
+    <!-- Rear wheel joints: velocity control -->
+    <joint name="rear_left_wheel_joint">
+      <command_interface name="velocity"/>
+      <state_interface name="position"/>
+      <state_interface name="velocity"/>
+    </joint>
+    <joint name="rear_right_wheel_joint">
+      <command_interface name="velocity"/>
+      <state_interface name="position"/>
+      <state_interface name="velocity"/>
+    </joint>
+  </ros2_control>
+  <!-- ========================= -->
+  <!-- GZ Sim ros2_control plugin -->
+  <!-- ========================= -->
+  <gazebo>
+    <plugin
+      filename="gz_ros2_control-system"
+      name="gz_ros2_control::GazeboSimROS2ControlPlugin">
+      <parameters>$(find mini_car_gazebo)/config/ros2_control.yaml</parameters>
+    </plugin>
+  </gazebo>
 </robot>

Commit message: update README

File: src/mini_car_description/urdf/mini_car.urdf.xacro (robot description, xacro)
@@ -160,5 +160,5 @@
     <origin xyz="0 0 0" rpy="0 0 0"/>
     <axis xyz="0 1 0"/>
-    <dynamics damping="0.1" friction="0.0"/>
+    <dynamics damping="0.1" friction="0.1"/>
   </joint>
   <!-- ========================= -->
@@ -297,6 +297,4 @@
     <kp>1000000.0</kp>
     <kd>100.0</kd>
-    <minDepth>0.001</minDepth>
-    <maxVel>0.1<maxVel>
   </gazebo>
   <gazebo reference="front_right_wheel_link">
@@ -306,6 +304,4 @@
     <kp>1000000.0</kp>
     <kd>100.0</kd>
-    <minDepth>0.001</minDepth>
-    <maxVel>0.1<maxVel>
   </gazebo>
   <gazebo reference="rear_left_wheel_link">
@@ -315,6 +311,4 @@
     <kp>1000000.0</kp>
     <kd>100.0</kd>
-    <minDepth>0.001</minDepth>
-    <maxVel>0.1<maxVel>
   </gazebo>
   <gazebo reference="rear_right_wheel_link">
@@ -324,6 +318,4 @@
     <kp>1000000.0</kp>
     <kd>100.0</kd>
-    <minDepth>0.001</minDepth>
-    <maxVel>0.1<maxVel>
   </gazebo>
   <gazebo reference="lidar_link">

Commit message: [FEAT]: add steering control (#6)
* add steering control

* ignore .home

* fix for test

* update README

File: src/mini_car_description/urdf/mini_car.urdf.xacro (robot description, xacro)
@@ -16,4 +16,9 @@
   <xacro:property name="lidar_radius" value="0.045"/>
   <xacro:property name="lidar_height" value="0.04"/>
+  <!-- Ackermann drive parameters -->
+  <xacro:property name="wheel_base" value="${front_axle_x - rear_axle_x}"/>
+  <xacro:property name="track_width" value="${wheel_y * 2.0}"/>
+  <xacro:property name="max_steer_angle" value="0.6"/>
+  <xacro:property name="max_speed" value="2.0"/>
   <!-- Derived values -->
   <xacro:property
@@ -147,5 +152,6 @@
     <origin xyz="${front_axle_x} ${wheel_y} ${wheel_joint_z}" rpy="0 0 0"/>
     <axis xyz="0 0 1"/>
-    <limit lower="-0.6" upper="0.6" effort="10.0" velocity="1.0"/>
+    <limit lower="${-max_steer_angle}" upper="${max_steer_angle}" effort="100.0" velocity="2.0"/>
+    <dynamics damping="1.0" friction="0.1"/>
   </joint>
   <joint name="front_left_wheel_joint" type="continuous">
@@ -154,4 +160,5 @@
     <origin xyz="0 0 0" rpy="0 0 0"/>
     <axis xyz="0 1 0"/>
+    <dynamics damping="0.1" friction="0.1"/>
   </joint>
   <!-- ========================= -->
@@ -165,5 +172,6 @@
     <origin xyz="${front_axle_x} ${-wheel_y} ${wheel_joint_z}" rpy="0 0 0"/>
     <axis xyz="0 0 1"/>
-    <limit lower="-0.6" upper="0.6" effort="10.0" velocity="1.0"/>
+    <limit lower="${-max_steer_angle}" upper="${max_steer_angle}" effort="100.0" velocity="2.0"/>
+    <dynamics damping="1.0" friction="0.1"/>
   </joint>
   <joint name="front_right_wheel_joint" type="continuous">
@@ -172,4 +180,5 @@
     <origin xyz="0 0 0" rpy="0 0 0"/>
     <axis xyz="0 1 0"/>
+    <dynamics damping="0.1" friction="0.0"/>
   </joint>
   <!-- ========================= -->
@@ -182,4 +191,5 @@
     <origin xyz="${rear_axle_x} ${wheel_y} ${wheel_joint_z}" rpy="0 0 0"/>
     <axis xyz="0 1 0"/>
+    <dynamics damping="0.1" friction="0.0"/>
   </joint>
   <!-- ========================= -->
@@ -192,4 +202,5 @@
     <origin xyz="${rear_axle_x} ${-wheel_y} ${wheel_joint_z}" rpy="0 0 0"/>
     <axis xyz="0 1 0"/>
+    <dynamics damping="0.1" friction="0.0"/>
   </joint>
   <!-- ========================= -->
@@ -230,3 +241,133 @@
       rpy="0 0 0"/>
   </joint>
+  <!-- ========================= -->
+  <!-- Virtual steering wheel -->
+  <!-- Used by gazebo_ros_ackermann_drive plugin -->
+  <!-- ========================= -->
+  <link name="steering_wheel_link">
+    <visual>
+      <origin xyz="0 0 0" rpy="1.5708 0 0"/>
+      <geometry>
+        <cylinder radius="0.04" length="0.01"/>
+      </geometry>
+      <material name="yellow"/>
+    </visual>
+    <collision>
+      <origin xyz="0 0 0" rpy="1.5708 0 0"/>
+      <geometry>
+        <cylinder radius="0.04" length="0.01"/>
+      </geometry>
+    </collision>
+    <inertial>
+      <origin xyz="0 0 0" rpy="0 0 0"/>
+      <mass value="0.05"/>
+      <inertia
+        ixx="0.00005"
+        ixy="0.0"
+        ixz="0.0"
+        iyy="0.00005"
+        iyz="0.0"
+        izz="0.00005"/>
+    </inertial>
+  </link>
+  <joint name="steering_wheel_joint" type="revolute">
+    <parent link="base_link"/>
+    <child link="steering_wheel_link"/>
+    <origin xyz="0.12 0 0.08" rpy="0 0 0"/>
+    <axis xyz="0 0 1"/>
+    <limit lower="-7.85" upper="7.85" effort="10.0" velocity="5.0"/>
+    <dynamics damping="0.1" friction="0.0"/>
+  </joint>
+  <!-- ========================= -->
+  <!-- Gazebo visual/friction properties -->
+  <!-- ========================= -->
+  <gazebo reference="base_link">
+    <material>Gazebo/Blue</material>
+  </gazebo>
+  <gazebo reference="front_left_steering_link">
+    <material>Gazebo/Yellow</material>
+  </gazebo>
+  <gazebo reference="front_right_steering_link">
+    <material>Gazebo/Yellow</material>
+  </gazebo>
+  <gazebo reference="front_left_wheel_link">
+    <material>Gazebo/Grey</material>
+    <mu1>1.5</mu1>
+    <mu2>1.5</mu2>
+    <kp>1000000.0</kp>
+    <kd>100.0</kd>
+  </gazebo>
+  <gazebo reference="front_right_wheel_link">
+    <material>Gazebo/Grey</material>
+    <mu1>1.5</mu1>
+    <mu2>1.5</mu2>
+    <kp>1000000.0</kp>
+    <kd>100.0</kd>
+  </gazebo>
+  <gazebo reference="rear_left_wheel_link">
+    <material>Gazebo/Grey</material>
+    <mu1>1.5</mu1>
+    <mu2>1.5</mu2>
+    <kp>1000000.0</kp>
+    <kd>100.0</kd>
+  </gazebo>
+  <gazebo reference="rear_right_wheel_link">
+    <material>Gazebo/Grey</material>
+    <mu1>1.5</mu1>
+    <mu2>1.5</mu2>
+    <kp>1000000.0</kp>
+    <kd>100.0</kd>
+  </gazebo>
+  <gazebo reference="lidar_link">
+    <material>Gazebo/Red</material>
+  </gazebo>
+  <gazebo reference="steering_wheel_link">
+    <material>Gazebo/Yellow</material>
+  </gazebo>
+  <!-- ========================= -->
+  <!-- ros2_control configuration -->
+  <!-- ========================= -->
+  <ros2_control name="GazeboSimSystem" type="system">
+    <hardware>
+      <plugin>gz_ros2_control/GazeboSimSystem</plugin>
+    </hardware>
+    <!-- Front steering joints: position control -->
+    <joint name="front_left_steering_joint">
+      <command_interface name="position">
+        <param name="min">-0.6</param>
+        <param name="max">0.6</param>
+      </command_interface>
+      <state_interface name="position"/>
+      <state_interface name="velocity"/>
+    </joint>
+    <joint name="front_right_steering_joint">
+      <command_interface name="position">
+        <param name="min">-0.6</param>
+        <param name="max">0.6</param>
+      </command_interface>
+      <state_interface name="position"/>
+      <state_interface name="velocity"/>
+    </joint>
+    <!-- Rear wheel joints: velocity control -->
+    <joint name="rear_left_wheel_joint">
+      <command_interface name="velocity"/>
+      <state_interface name="position"/>
+      <state_interface name="velocity"/>
+    </joint>
+    <joint name="rear_right_wheel_joint">
+      <command_interface name="velocity"/>
+      <state_interface name="position"/>
+      <state_interface name="velocity"/>
+    </joint>
+  </ros2_control>
+  <!-- ========================= -->
+  <!-- GZ Sim ros2_control plugin -->
+  <!-- ========================= -->
+  <gazebo>
+    <plugin
+      filename="gz_ros2_control-system"
+      name="gz_ros2_control::GazeboSimROS2ControlPlugin">
+      <parameters>$(find mini_car_gazebo)/config/ros2_control.yaml</parameters>
+    </plugin>
+  </gazebo>
 </robot>
