Commit message: add rviz-gazebo simulation

File: src/mini_car_description/urdf/mini_car.urdf.xacro (robot description, xacro)
@@ -282,15 +282,5 @@
   <!-- Gazebo visual/friction properties -->
   <!-- ========================= -->
-  <gazebo reference="base_link">
-    <material>Gazebo/Blue</material>
-  </gazebo>
-  <gazebo reference="front_left_steering_link">
-    <material>Gazebo/Yellow</material>
-  </gazebo>
-  <gazebo reference="front_right_steering_link">
-    <material>Gazebo/Yellow</material>
-  </gazebo>
   <gazebo reference="front_left_wheel_link">
-    <material>Gazebo/Grey</material>
     <mu1>1.5</mu1>
     <mu2>1.5</mu2>
@@ -299,5 +289,4 @@
   </gazebo>
   <gazebo reference="front_right_wheel_link">
-    <material>Gazebo/Grey</material>
     <mu1>1.5</mu1>
     <mu2>1.5</mu2>
@@ -306,5 +295,4 @@
   </gazebo>
   <gazebo reference="rear_left_wheel_link">
-    <material>Gazebo/Grey</material>
     <mu1>1.5</mu1>
     <mu2>1.5</mu2>
@@ -313,15 +301,8 @@
   </gazebo>
   <gazebo reference="rear_right_wheel_link">
-    <material>Gazebo/Grey</material>
     <mu1>1.5</mu1>
     <mu2>1.5</mu2>
     <kp>1000000.0</kp>
     <kd>100.0</kd>
-  </gazebo>
-  <gazebo reference="lidar_link">
-    <material>Gazebo/Red</material>
-  </gazebo>
-  <gazebo reference="steering_wheel_link">
-    <material>Gazebo/Yellow</material>
   </gazebo>
   <!-- ========================= -->

Commit message: [FEAT]: add rviz-gazebo simulation (#7)
* add rviz-gazebo simulation

File: src/mini_car_description/urdf/mini_car.urdf.xacro (robot description, xacro)
@@ -282,15 +282,5 @@
   <!-- Gazebo visual/friction properties -->
   <!-- ========================= -->
-  <gazebo reference="base_link">
-    <material>Gazebo/Blue</material>
-  </gazebo>
-  <gazebo reference="front_left_steering_link">
-    <material>Gazebo/Yellow</material>
-  </gazebo>
-  <gazebo reference="front_right_steering_link">
-    <material>Gazebo/Yellow</material>
-  </gazebo>
   <gazebo reference="front_left_wheel_link">
-    <material>Gazebo/Grey</material>
     <mu1>1.5</mu1>
     <mu2>1.5</mu2>
@@ -299,5 +289,4 @@
   </gazebo>
   <gazebo reference="front_right_wheel_link">
-    <material>Gazebo/Grey</material>
     <mu1>1.5</mu1>
     <mu2>1.5</mu2>
@@ -306,5 +295,4 @@
   </gazebo>
   <gazebo reference="rear_left_wheel_link">
-    <material>Gazebo/Grey</material>
     <mu1>1.5</mu1>
     <mu2>1.5</mu2>
@@ -313,15 +301,8 @@
   </gazebo>
   <gazebo reference="rear_right_wheel_link">
-    <material>Gazebo/Grey</material>
     <mu1>1.5</mu1>
     <mu2>1.5</mu2>
     <kp>1000000.0</kp>
     <kd>100.0</kd>
-  </gazebo>
-  <gazebo reference="lidar_link">
-    <material>Gazebo/Red</material>
-  </gazebo>
-  <gazebo reference="steering_wheel_link">
-    <material>Gazebo/Yellow</material>
   </gazebo>
   <!-- ========================= -->
@@ -349,4 +330,13 @@
       <state_interface name="velocity"/>
     </joint>
+    <!-- Passive front wheel joints: expose state so robot_state_publisher can complete the TF tree. -->
+    <joint name="front_left_wheel_joint">
+      <state_interface name="position"/>
+      <state_interface name="velocity"/>
+    </joint>
+    <joint name="front_right_wheel_joint">
+      <state_interface name="position"/>
+      <state_interface name="velocity"/>
+    </joint>
     <!-- Rear wheel joints: velocity control -->
     <joint name="rear_left_wheel_joint">
@@ -357,4 +347,8 @@
     <joint name="rear_right_wheel_joint">
       <command_interface name="velocity"/>
+      <state_interface name="position"/>
+      <state_interface name="velocity"/>
+    </joint>
+    <joint name="steering_wheel_joint">
       <state_interface name="position"/>
       <state_interface name="velocity"/>

Commit message: add Lidar simulation

File: src/mini_car_description/urdf/mini_car.urdf.xacro (robot description, xacro)
@@ -15,5 +15,5 @@
   <xacro:property name="wheel_y" value="0.17"/>
   <xacro:property name="lidar_radius" value="0.045"/>
-  <xacro:property name="lidar_height" value="0.04"/>
+  <xacro:property name="lidar_height" value="0.1"/>
   <!-- Ackermann drive parameters -->
   <xacro:property name="wheel_base" value="${front_axle_x - rear_axle_x}"/>
@@ -205,6 +205,5 @@
   </joint>
   <!-- ========================= -->
-  <!-- LiDAR placeholder -->
-  <!-- The actual Gazebo LiDAR sensor will be added later. -->
+  <!-- LiDAR -->
   <!-- ========================= -->
   <link name="lidar_link">
@@ -241,4 +240,27 @@
       rpy="0 0 0"/>
   </joint>
+  <gazebo reference="lidar_link">
+    <sensor name="lidar_sensor" type="gpu_lidar">
+      <topic>/scan</topic>
+      <update_rate>10</update_rate>
+      <lidar>
+        <scan>
+          <horizontal>
+            <samples>720</samples>
+            <resolution>1</resolution>
+            <min_angle>-2.35619449</min_angle>
+            <max_angle>2.35619449</max_angle>
+          </horizontal>
+        </scan>
+        <range>
+          <min>0.08</min>
+          <max>8.0</max>
+          <resolution>0.01</resolution>
+        </range>
+      </lidar>
+      <always_on>true</always_on>
+      <visualize>true</visualize>
+    </sensor>
+  </gazebo>
   <!-- ========================= -->
   <!-- Virtual steering wheel -->
